File: LMR33640/24to5-lmr33640.kicad_sch (KiCad schematic)
At the start: 14 parts, among them J1 Conn_01x02, U1 LMR33640ADDA

Commit message: layout done
Parts:
- added C5: 100uF 35V, Capacitor_THT:CP_Radial_D6.3mm_P2.50mm, symbol Device:C_Polarized
- added C6, C7: 22uF, Capacitor_SMD:C_1206_3216Metric, symbol Device:C
- added D2: SMAJ28A, Diode_SMD:D_SMA, symbol Diode:SM6T27A
- added D3: SMAJ5.0A, Diode_SMD:D_SMA, symbol Diode:SM6T27A
- added D4: LED, LED_SMD:LED_0603_1608Metric, symbol Device:LED
- added J2: USB_C_Receptacle_PowerOnly_6P, TYPE-C-31-M-17:TYPEC31M17, symbol Connector:USB_C_Receptacle_PowerOnly_6P
- added R4, R5: 10k, Resistor_SMD:R_0603_1608Metric, symbol Device:R
- added R6: 100k, Resistor_SMD:R_0603_1608Metric, symbol Device:R
- J1: footprint Connector_AMASS:AMASS_XT30PW-M_1x02_P2.50mm_Horizontal -> Connector_AMASS:AMASS_XT30U-M_1x02_P5.0mm_Vertical
Connections:
- net +24V: now also C6.1, D2.1 (A1), R6.1
- net GND: now also TP2.1, C5.2, C6.2, C7.2, D2.2 (A2), D3.2 (A2), D4.1 (K), J2.A12 (GND), J2.B12 (GND), J2.S1 (SHIELD)
- net +5V: now reaches C1.1, L1.2, R1.1
- net +5V: now also TP1.1, C5.1, C7.1, D3.1 (A1), J2.A9 (VBUS), J2.B9 (VBUS), R4.2, R5.2
- new net: D4.2 (A), R6.2
- new net: J2.B5 (CC2), R5.1
- new net: J2.A5 (CC1), R4.1
Other:
- moved on the sheet: C4, F1, J1
