File: LMR33640/24to5-lmr33640.kicad_pcb (KiCad board)
At the start: 2 copper layers, 20 x 37 mm, 24 parts, among them J1 Conn_01x02, J2 USB_C_Receptacle_PowerOnly_6P, U1 LMR33640ADDA

Commit message: decoration
Parts:
- moved C1 2.29 mm to (78.0, 82.7), turned to 90 degrees
- moved R1 2.29 mm to (75.7, 82.7), turned to 0 degrees
Routing:
- net GND: vias 2 -> 29
Other:
- board text added: "+5V"
- board text added: "GND"
- board text added: "JLCJLCJLCJLC"
- board text added: "Output 5V4A"
- board text added: "USB 5V PowerSupply"
- board text added: "by RY ver.1.0"
